File: pcb/mikroproje.kicad_pcb (KiCad board)
At the start: 2 copper layers, 132.8 x 58.5 mm, 28 parts, among them J1 Conn_01x02, J2 Conn_01x02, Q1 BC817, SW1 SW_Push, U1 MSP430G2553IN20, U2 OLED, U3 HC-05, U4 TJ7533AGF, U5 MPU6050

Commit message: Update revised portable posture analyzer PCB files
Parts:
- removed Q1: BC817, Package_TO_SOT_SMD:SOT-23
- added Q2: MMBT2222A, Package_TO_SOT_SMD:SOT-23, F.Cu at (63.2, 131.4)
- C5: value 1uF -> 2.2uF
- U4: value TJ7533AGF -> ap2210n-3.3trg1; footprint Package_TO_SOT_SMD:SOT-89-3 -> Package_TO_SOT_SMD:SOT-23-3
- moved D4 4.73 mm to (57.4, 98.0)
- moved R4 2.66 mm to (51.5, 98.0)
- moved C5 0.69 mm to (51.6, 105.1)
- moved U4 0.30 mm to (47.2, 104.8)
Connections:
- J1 pad 1: Vbat -> Vbat_in
- R6 pad 1: Vbat -> Vbat_in
- U4 pad 2: Vbat_in -> 3V3
- U4 pad 3: 3V3 -> Vbat_in
Routing:
- net Vbat_in: track 51.6 -> 48.7 mm
- net Net-(D4-A): track 3.73 -> 5.81 mm
- net Net-(D2-A): track 30.8 -> 32.4 mm
