File: pcb/mikroproje.kicad_sch (KiCad schematic)
At the start: 28 parts, among them J1 Conn_01x02, J2 Conn_01x02, Q1 BC817, SW1 SW_Push, U1 MSP430G2553IN20, U2 OLED, U3 HC-05, U4 TJ7533AGF, U5 MPU6050

Commit message: Update revised portable posture analyzer PCB files
Parts:
- removed D3: D_Schottky, Diode_SMD:D_SOD-123, symbol Device:D_Schottky
- removed Q1: BC817, Package_TO_SOT_SMD:SOT-23, symbol Transistor_BJT:BC817
- removed U4: TJ7533AGF, Package_TO_SOT_SMD:SOT-89-3, symbol 1_Modules:TJ7533AGF
- added Q2: MMBT2222A, Package_TO_SOT_SMD:SOT-23, symbol Transistor_BJT:MMBT2222A
- added U4: ap2210n-3.3trg1, Package_TO_SOT_SMD:SOT-23-3, symbol 1_Modules:ap2210n-3.3trg1
- C5: value 1uF -> 2.2uF
Connections:
- net Vbat_in is gone; now on net Vbat: C2.1, U3.5 (5V)
- net 3V3: now also U4.2 (Vout)
- net GND: now also Q2.2 (E), U4.1 (GND)
- net Vbat: now also U4.3 (Vin)
- net at R10.1, R2.2: now also Q2.1 (B)
- net at C6.2, D2.2 (A), J2.2 (Pin_2): now also Q2.3 (C)
Other:
- note removed: "100mA"
- moved on the sheet: C2, C5
